File: PCB/LightTable.kicad_pcb (KiCad board)
At the start: 2 copper layers, 18 parts, among them CON1 BARREL_JACK, P1 CONN_2_V, P2 CONN_01X01, P3 CONN_01X01, P4 CONN_01X01, P5 CONN_01X01, P6 CONN_01X01, P7 CONN_01X01, P8 CONN_4_V, U1 MosfetIRF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

Commit message: Added Power Led and BOM
Parts:
- added D1: PWR, LEDs:LED-5MM, B.Cu at (123.8, 90.2)
- added R2: 330, Resistors_ThroughHole:Resistor_Horizontal_RM10mm, B.Cu at (131.4, 85.1)
- renumbered SHIELD1 to Led_Strip_Driver-shield
Routing:
- net Net-(D1-Pad1): track 0.00 -> 7.62 mm
- net V5: track 29.5 -> 36.5 mm
Changed lines of the file:
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@@
 (kicad_pcb (version 4) (host pcbnew "(2015-07-07 BZR 5906)-product")
   (general
-    (links 36)
+    (links 39)
     (no_connects 1)
     (area 0 0 0 0)
     (thickness 1.6)
     (drawings 0)
-    (tracks 74)
+    (tracks 76)
     (zones 0)
-    (modules 18)
-    (nets 31)
+    (modules 20)
+    (nets 32)
   )
   (page A4)
@@
   (net 29 PWM_B)
   (net 30 PWM_G)
+  (net 31 "Net-(D1-Pad1)")
   (net_class Default "This is the default net class."
     (clearance 0.635)
@@
     (add_net G)
     (add_net GND)
+    (add_net "Net-(D1-Pad1)")
     (add_net R)
     (add_net V5)
@@
   (module arduino_shields:ARDUINO_SHIELD_2_040pins (layer F.Cu)
     (at 72.39 104.14)
-    (fp_text reference SHIELD1 (at 5.715 -57.15) (layer F.SilkS)
+    (fp_text reference Led_Strip_Driver-shield (at 13.335 -56.515) (layer F.SilkS)
       (effects (font (thickness 0.3048)))
     )
@@
     )
   )
+  (module LEDs:LED-5MM (layer B.Cu)
+    (at 123.825 90.17 180)
+    (descr "LED 5mm round vertical")
+    (tags "LED 5mm round vertical")
+    (fp_text reference D1 (at 1.524 -4.064 180) (layer B.SilkS)
+      (effects (font (size 1 1) (thickness 0.15)) (justify mirror))
+    )
+    (fp_text value PWR (at 1.524 3.937 180) (layer B.Fab)
+      (effects (font (size 1 1) (thickness 0.15)) (justify mirror))
+    )
+    (fp_line (start -1.5 1.55) (end -1.5 -1.55) (layer B.CrtYd) (width 0.05))
+    (fp_arc (start 1.3 0) (end -1.5 -1.55) (angle 302) (layer B.CrtYd) (width 0.05))
+    (fp_arc (start 1.27 0) (end -1.23 1.5) (angle -297.5) (layer B.SilkS) (width 0.15))
+    (fp_line (start -1.23 -1.5) (end -1.23 1.5) (layer B.SilkS) (width 0.15))
+    (fp_circle (center 1.27 0) (end 0.97 2.5) (layer B.SilkS) (width 0.15))
+    (fp_text user K (at -1.905 -1.905 180) (layer B.SilkS)
+      (effects (font (size 1 1) (thickness 0.15)) (justify mirror))
+    )
+    (pad 1 thru_hole rect (at 0 0 90) (size 2 1.9) (drill 1.00076) (layers *.Cu *.Mask B.SilkS)
+      (net 31 "Net-(D1-Pad1)"))
+    (pad 2 thru_hole circle (at 2.54 0 180) (size 1.9 1.9) (drill 1.00076) (layers *.Cu *.Mask B.SilkS)
+      (net 3 V5))
+    (model LEDs.3dshapes/LED-5MM.wrl
+      (at (xyz 0.05 0 0))
+      (scale (xyz 1 1 1))
+      (rotate (xyz 0 0 90))
+    )
+  )
+  (module Resistors_ThroughHole:Resistor_Horizontal_RM10mm (layer B.Cu)
+    (at 131.445 85.09 90)
+    (descr "Resistor, Axial,  RM 10mm, 1/3W,")
+    (tags "Resistor, Axial, RM 10mm, 1/3W,")
+    (fp_text reference R2 (at 0.24892 3.50012 90) (layer B.SilkS)
+      (effects (font (size 1 1) (thickness 0.15)) (justify mirror))
+    )
+    (fp_text value 330 (at 3.81 -3.81 90) (layer B.Fab)
+      (effects (font (size 1 1) (thickness 0.15)) (justify mirror))
+    )
+    (fp_line (start -2.54 1.27) (end 2.54 1.27) (layer B.SilkS) (width 0.15))
+    (fp_line (start 2.54 1.27) (end 2.54 -1.27) (layer B.SilkS) (width 0.15))
+    (fp_line (start 2.54 -1.27) (end -2.54 -1.27) (layer B.SilkS) (width 0.15))
+    (fp_line (start -2.54 -1.27) (end -2.54 1.27) (layer B.SilkS) (width 0.15))
+    (fp_line (start -2.54 0) (end -3.81 0) (layer B.SilkS) (width 0.15))
+    (fp_line (start 2.54 0) (end 3.81 0) (layer B.SilkS) (width 0.15))
+    (pad 1 thru_hole circle (at -5.08 0 90) (size 1.99898 1.99898) (drill 1.00076) (layers *.Cu *.SilkS *.Mask)
+      (net 31 "Net-(D1-Pad1)"))
+    (pad 2 thru_hole circle (at 5.08 0 90) (size 1.99898 1.99898) (drill 1.00076) (layers *.Cu *.SilkS *.Mask)
+      (net 1 GND))
+    (model Resistors_ThroughHole.3dshapes/Resistor_Horizontal_RM10mm.wrl
+      (at (xyz 0 0 0))
+      (scale (xyz 0.4 0.4 0.4))
+      (rotate (xyz 0 0 0))
+    )
+  )
   (segment (start 92.71 90.17) (end 92.71 86.995) (width 1.524) (layer F.Cu) (net 2))
   (segment (start 92.71 86.995) (end 90.805 85.09) (width 1.524) (layer F.Cu) (net 2))
@@
   (segment (start 93.472 97.282) (end 93.472 99.06) (width 1.524) (layer F.Cu) (net 2))
   (segment (start 92.71 96.52) (end 93.472 97.282) (width 1.524) (layer F.Cu) (net 2))
+  (segment (start 121.285 90.17) (end 114.3 90.17) (width 1.016) (layer F.Cu) (net 3) (status 400000))
   (segment (start 97.79 90.17) (end 114.3 90.17) (width 1.016) (layer F.Cu) (net 3))
   (segment (start 115.276 91.146) (end 115.276 93.726) (width 1.016) (layer F.Cu) (net 3))
@@
   (segment (start 95.25 66.04) (end 107.315 66.04) (width 0.762) (layer F.Cu) (net 30))
   (segment (start 93.98 67.31) (end 95.25 66.04) (width 0.762) (layer F.Cu) (net 30))
+  (segment (start 123.825 90.17) (end 131.445 90.17) (width 1.016) (layer F.Cu) (net 31) (status C00000))
   (zone (net 1) (net_name GND) (layer F.Cu) (hatch edge 0.508)
     (connect_pads (clearance 0.508))
