File: PCB/LightTable.kicad_pcb (KiCad board)
At the start: 2 copper layers, 20 parts, among them CON1 BARREL_JACK, P1 CONN_2_V, P2 CONN_01X01, P3 CONN_01X01, P4 CONN_01X01, P5 CONN_01X01, P6 CONN_01X01, P7 CONN_01X01, P8 CONN_4_V, U1 MosfetIRF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

Commit message: Changed capacitor values
Parts:
- moved C1 14.1 mm to (111.8, 87.0)
Routing:
- net +12V: track 44.8 -> 59.6 mm
Changed lines of the file:
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@@
     (thickness 1.6)
     (drawings 0)
-    (tracks 76)
+    (tracks 79)
     (zones 0)
     (modules 20)
@@
   )
   (module Capacitors_ThroughHole:C_Disc_D3_P2.5 (layer B.Cu)
-    (at 97.79 85.09 180)
+    (at 111.76 86.995 180)
     (descr "Capacitor 3mm Disc, Pitch 2.5mm")
     (tags Capacitor)
@@
     )
   )
+  (segment (start 109.26 86.995) (end 103.505 86.995) (width 1.524) (layer F.Cu) (net 2) (status 400000))
+  (segment (start 95.29 85.09) (end 90.805 85.09) (width 1.524) (layer F.Cu) (net 2))
+  (segment (start 101.6 85.09) (end 95.29 85.09) (width 1.524) (layer F.Cu) (net 2))
+  (segment (start 103.505 86.995) (end 101.6 85.09) (width 1.524) (layer F.Cu) (net 2))
   (segment (start 92.71 90.17) (end 92.71 86.995) (width 1.524) (layer F.Cu) (net 2))
   (segment (start 92.71 86.995) (end 90.805 85.09) (width 1.524) (layer F.Cu) (net 2))
@@
   (segment (start 89.535 85.09) (end 90.805 85.09) (width 1.524) (layer F.Cu) (net 2))
   (segment (start 89.535 85.09) (end 86.19 85.09) (width 1.524) (layer F.Cu) (net 2))
-  (segment (start 90.805 85.09) (end 95.29 85.09) (width 1.524) (layer F.Cu) (net 2) (status 2))
   (segment (start 92.71 90.17) (end 92.71 96.52) (width 1.524) (layer F.Cu) (net 2))
   (segment (start 93.472 97.282) (end 93.472 99.06) (width 1.524) (layer F.Cu) (net 2))

Commit message: Added led for showing when a long click has been made
Parts:
- removed Led_Strip_Driver-shield: ARDUINO_SHIELD, arduino_shields:ARDUINO_SHIELD_2_040pins
- added D2: Long, LEDs:LED-5MM, B.Cu at (116.2, 67.3)
- added R3: 330, Resistors_ThroughHole:Resistor_Horizontal_RM10mm, B.Cu at (116.8, 81.9)
- added SHIELD1: ARDUINO_SHIELD, arduino_shields:ARDUINO_SHIELD_2_040pins, F.Cu at (72.4, 104.1)
- moved R1 4.26 mm to (135.3, 85.1)
- moved P2 1.91 mm to (105.4, 59.7)
- moved P3 1.91 mm to (114.9, 59.7)
Routing:
- net Net-(D2-Pad2): track 0.00 -> 12.2 mm
- net Net-(D2-Pad1): track 0.00 -> 11.4 mm
- net PBtn: track 36.7 -> 34.6 mm
